File: hardware/odsk.sch (KiCad schematic (older format))
At the start: 28 parts, among them J1 AudioJack4, J2 Raspberry_Pi_Zero, U1 TPS73133DBV, U2 PCM5102

Commit message: update cap footprint
Parts:
- C3: footprint Capacitor_SMD:C_0805_2012Metric_Pad1.18x1.45mm_HandSolder -> Capacitor_SMD:C_1206_3216Metric_Pad1.33x1.80mm_HandSolder
Changed lines of the file:
@@
 F 0 "C3" H 3158 1696 50  0000 R CNN
 F 1 "100u" H 3158 1605 50  0000 R CNN
-F 2 "Capacitor_SMD:C_0805_2012Metric_Pad1.18x1.45mm_HandSolder" H 3250 1650 50  0001 C CNN
+F 2 "Capacitor_SMD:C_1206_3216Metric_Pad1.33x1.80mm_HandSolder" H 3250 1650 50  0001 C CNN
 F 3 "~" H 3250 1650 50  0001 C CNN
 	1    3250 1650
